File: mallory.kicad_pcb (KiCad board)
At the start: 2 copper layers, 130 parts, among them SW1 SW_PUSH, SW10 SW_PUSH, SW11 SW_PUSH, SW12 SW_PUSH, SW13 SW_PUSH, SW14 SW_PUSH, SW15 SW_PUSH, SW16 SW_PUSH, SW17 SW_PUSH, SW18 SW_PUSH, SW19 SW_PUSH, SW2 SW_PUSH, SW20 SW_PUSH, SW21 SW_PUSH, SW22 SW_PUSH, SW23 SW_PUSH, SW24 SW_PUSH, SW25 SW_PUSH, SW26 SW_PUSH, SW27 SW_PUSH, SW28 SW_PUSH, SW29 SW_PUSH, SW3 SW_PUSH, SW30 SW_PUSH, SW31 SW_PUSH, SW32 SW_PUSH, SW33 SW_PUSH, SW34 SW_PUSH, SW35 SW_PUSH, SW36 SW_PUSH, SW37 SW_PUSH, SW38 SW_PUSH, SW39 SW_PUSH, SW4 SW_PUSH, SW40 SW_PUSH, SW41 SW_PUSH, SW42 SW_PUSH, SW43 SW_PUSH, SW44 SW_PUSH, SW45 SW_PUSH, SW46 SW_PUSH, SW47 SW_PUSH, SW48 SW_PUSH, SW49 SW_PUSH, SW5 SW_PUSH, SW50 SW_PUSH, SW51 SW_PUSH, SW52 SW_PUSH, SW53 SW_PUSH, SW54 SW_PUSH, SW55 SW_PUSH, SW56 SW_PUSH, SW57 SW_PUSH, SW58 SW_PUSH, SW59 SW_PUSH, SW6 SW_PUSH, SW60 SW_PUSH, SW61 SW_PUSH, SW62 SW_PUSH, SW63 SW_PUSH, SW64 SW_PUSH, SW65 SW_PUSH, SW7 SW_PUSH, SW8 SW_PUSH, SW9 SW_PUSH, U1 ProMicro

Commit message: Update
Parts:
- added D65: D, kbd:D3_TH, F.Cu at (375.5, 145.5)
- added SW33B1: SW_PUSH, MXOnly:MXOnly-1U-NoLED, F.Cu at (81.2, 107.3)
- added SW64B1: SW_PUSH, MXOnly:MXOnly-2U-ReversedStabilizers-NoLED, F.Cu at (166.4, 153.4)
- added SW65B1: SW_PUSH, MXOnly:MXOnly-1.25U-NoLED, F.Cu at (196.7, 159.8)
- added SW66: SW_PUSH, MXOnly:MXOnly-1.25U-NoLED, F.Cu at (366.6, 145.5)
- D1, D10, D11, D12, D13, D14, D15, D16, D17, D18, D19, D2, D20, D21, D22, D23, D24, D25, D26, D27, D28, D29, D3, D30, D31, D32, D33, D34, D35, D36, D37, D38, D39, D4, D40, D41, D42, D43, D44, D45, D46, D47, D48, D49, D5, D50, D51, D52, D53, D54, D55, D56, D57, D58, D59, D6, D60, D61, D62, D63, D64, D7, D8, D9: footprint kbd:D3_TH_SMD -> kbd:D3_TH
- SW10, SW11, SW12, SW13, SW14, SW17, SW19, SW2, SW20, SW23, SW24, SW25, SW26, SW27, SW28, SW29, SW3, SW30, SW32, SW34, SW35, SW36, SW37, SW38, SW39, SW4, SW40, SW41, SW42, SW43, SW44, SW47, SW48, SW49, SW5, SW51, SW52, SW53, SW54, SW55, SW59: footprint MXOnly:MXOnly-1U-Hotswap -> MXOnly:MXOnly-1U-NoLED
- SW15, SW6: footprint MXOnly:MXOnly-1.5U-Hotswap -> MXOnly:MXOnly-1U-NoLED
- SW16: footprint MXOnly:MXOnly-2.25U-Hotswap-ReversedStabilizers -> MXOnly:MXOnly-2U-NoLED
- SW18, SW31: footprint MXOnly:MXOnly-1U-Hotswap -> MXOnly:MXOnly-1.5U-NoLED
- SW21: footprint MXOnly:MXOnly-1U-leftleg -> MXOnly:MXOnly-1U-NoLED
- SW22: footprint MXOnly:MXOnly-1U-rightleg -> MXOnly:MXOnly-1U-NoLED
- SW33, SW58: footprint MXOnly:MXOnly-1U-Hotswap -> MXOnly:MXOnly-1.75U-NoLED
- SW45: footprint MXOnly:MXOnly-1U-Hotswap -> MXOnly:MXOnly-2.25U-ReversedStabilizers-NoLED
- SW46: footprint MXOnly:MXOnly-1U-Hotswap -> MXOnly:MXOnly-2.25U-NoLED
- SW50: footprint MXOnly:MXOnly-2U-Hotswap -> MXOnly:MXOnly-1U-NoLED
- SW56, SW65, SW9: footprint MXOnly:MXOnly-1.25U-Hotswap -> MXOnly:MXOnly-1U-NoLED
- SW57: footprint MXOnly:MXOnly-2.75U-Hotswap-ReversedStabilizers -> MXOnly:MXOnly-1U-NoLED
- SW60: footprint MXOnly:MXOnly-1.5U-Hotswap -> MXOnly:MXOnly-1.25U-NoLED
- SW61: footprint MXOnly:MXOnly-1U-Hotswap -> MXOnly:MXOnly-2.75U-ReversedStabilizers-NoLED
- SW62: footprint MXOnly:MXOnly-2.25U-Hotswap-ReversedStabilizers -> MXOnly:MXOnly-1.25U-NoLED
- SW63: footprint MXOnly:MXOnly-1U-Hotswap -> MXOnly:MXOnly-1.25U-NoLED
- SW64: footprint MXOnly:MXOnly-2.75U-Hotswap -> MXOnly:MXOnly-2.25U-ReversedStabilizers-NoLED
- SW7: footprint MXOnly:MXOnly-1.75U-Hotswap -> MXOnly:MXOnly-1U-NoLED
- SW8: footprint MXOnly:MXOnly-2.25U-Hotswap -> MXOnly:MXOnly-1U-NoLED
- U1: moved to B.Cu
- moved SW60 288.2 mm to (79.4, 145.4)
- moved D59 282.5 mm to (88.0, 145.8), turned to 90 degrees
- moved SW62 229.3 mm to (133.3, 147.9), turned to 348 degrees
- moved D61 227.5 mm to (141.7, 150.1), turned to 78 degrees
- moved D14 208.3 mm to (332.6, 69.1), turned to 90 degrees
- moved SW15 206.8 mm to (324.4, 69.2), turned to 0 degrees
- moved D15 206.6 mm to (370.6, 69.3), turned to 90 degrees
- moved SW32 205.7 mm to (55.8, 105.2), turned to 0 degrees
- moved SW16 202.6 mm to (353.0, 69.2), turned to 0 degrees
- moved D31 200.2 mm to (64.0, 105.0), turned to 90 degrees
- moved D13 198.5 mm to (313.8, 66.8)
- moved SW14 197.4 mm to (305.8, 67.1)
- moved SW33 194.9 mm to (85.8, 107.2), turned to 0 degrees
- moved SW64 191.7 mm to (168.7, 154.0), turned to 348 degrees
- moved D49 190.7 mm to (183.3, 137.6), turned to 78 degrees
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Connections:
- D16 pad 1: row1 -> row2
- D23 pad 1: row2 -> row3
- D24 pad 1: row2 -> row3
- D31 pad 1: row3 -> row4
- D32 pad 1: row3 -> row4
- D38 pad 1: row4 -> row5
- D39 pad 1: row4 -> row5
- D40 pad 1: row4 -> row5
- D45 pad 1: row5 -> row6
- D46 pad 1: row5 -> row6
- D47 pad 1: row5 -> row6
- D48 pad 1: row5 -> row6
- D51 pad 1: row6 -> row7
- D52 pad 1: row6 -> row7
- D53 pad 1: row6 -> row7
- D54 pad 1: row6 -> row7
- D55 pad 1: row6 -> row7
- D56 pad 1: row6 -> row7
- D59 pad 1: row7 -> row8
- D60 pad 1: row7 -> row8
- D61 pad 1: row7 -> row8
- D62 pad 1: row7 -> row8
- D63 pad 1: row7 -> row8
- D64 pad 1: row7 -> row8
- SW10 pad 1: Net-(SW10-Pad1) -> col0
- SW12 pad 1: Net-(SW12-Pad1) -> col2
- SW13 pad 1: Net-(SW13-Pad1) -> col3
- SW17 pad 1: col7 -> col0
- SW18 pad 1: Net-(SW10-Pad1) -> col1
- SW19 pad 1: col1 -> col2
- SW2 pad 1: Net-(SW10-Pad1) -> col0
- SW20 pad 1: Net-(SW12-Pad1) -> col3
- SW21 pad 1: Net-(SW13-Pad1) -> col4
- SW22 pad 1: col4 -> col5
- SW23 pad 1: col5 -> col6
- SW24 pad 1: col6 -> col0
- SW25 pad 1: col7 -> col1
- SW26 pad 1: Net-(SW10-Pad1) -> col2
- SW27 pad 1: col1 -> col3
- SW28 pad 1: Net-(SW12-Pad1) -> col4
- SW29 pad 1: Net-(SW13-Pad1) -> col5
- SW30 pad 1: col4 -> col6
- SW31 pad 1: col5 -> col7
- SW32 pad 1: col6 -> col0
- SW33 pad 1: col7 -> col1
- SW34 pad 1: Net-(SW10-Pad1) -> col2
- SW35 pad 1: col1 -> col3
- SW36 pad 1: Net-(SW12-Pad1) -> col4
- SW37 pad 1: Net-(SW13-Pad1) -> col5
- SW38 pad 1: col4 -> col6
- SW39 pad 1: col5 -> col0
- SW4 pad 1: Net-(SW12-Pad1) -> col2
- SW40 pad 1: col6 -> col1
- SW41 pad 1: col7 -> col2
- SW42 pad 1: Net-(SW10-Pad1) -> col3
- SW43 pad 1: col1 -> col4
- SW44 pad 1: Net-(SW12-Pad1) -> col5
- SW45 pad 1: Net-(SW13-Pad1) -> col6
- SW46 pad 1: col4 -> col1
- SW47 pad 1: col5 -> col2
- SW48 pad 1: col6 -> col3
- SW49 pad 1: col7 -> col4
- SW5 pad 1: Net-(SW13-Pad1) -> col3
- SW50 pad 1: Net-(SW10-Pad1) -> col5
- SW51 pad 1: col1 -> col6
- SW52 pad 1: Net-(SW12-Pad1) -> col0
- SW53 pad 1: Net-(SW13-Pad1) -> col1
- SW54 pad 1: col4 -> col2
- SW55 pad 1: col5 -> col3
- SW56 pad 1: col6 -> col4
- SW57 pad 1: col7 -> col5
- SW58 pad 1: Net-(SW10-Pad1) -> col6
- SW59 pad 1: col1 -> col7
- SW60 pad 1: Net-(SW12-Pad1) -> col0
- SW61 pad 1: Net-(SW13-Pad1) -> col1
- SW62 pad 1: col4 -> col2
- SW63 pad 1: col5 -> col3
- SW64 pad 1: col6 -> col5
- SW65 pad 1: col7 -> col6
- U1 pad 10: row5 -> row4
- U1 pad 12: row7 -> row8
- U1 pad 13: col7 -> row7
- U1 pad 14: col6 -> row5
- U1 pad 15: col5 -> row3
- U1 pad 16: col4 -> row1
- U1 pad 2: Net-(U1-Pad2) -> col4
- U1 pad 5: row0 -> col5
- U1 pad 6: row1 -> col6
- U1 pad 7: row2 -> col7
- U1 pad 8: row3 -> row0
- U1 pad 9: row4 -> row2
Other:
- board outline added: 337.5 x 116.5 mm
