File: mallory.sch (KiCad schematic (older format))
At the start: 130 parts, among them SW1 SW_PUSH, SW10 SW_PUSH, SW11 SW_PUSH, SW12 SW_PUSH, SW13 SW_PUSH, SW14 SW_PUSH, SW15 SW_PUSH, SW16 SW_PUSH, SW17 SW_PUSH, SW18 SW_PUSH, SW19 SW_PUSH, SW2 SW_PUSH, SW20 SW_PUSH, SW21 SW_PUSH, SW22 SW_PUSH, SW23 SW_PUSH, SW24 SW_PUSH, SW25 SW_PUSH, SW26 SW_PUSH, SW27 SW_PUSH, SW28 SW_PUSH, SW29 SW_PUSH, SW3 SW_PUSH, SW30 SW_PUSH, SW31 SW_PUSH, SW32 SW_PUSH, SW33 SW_PUSH, SW34 SW_PUSH, SW35 SW_PUSH, SW36 SW_PUSH, SW37 SW_PUSH, SW38 SW_PUSH, SW39 SW_PUSH, SW4 SW_PUSH, SW40 SW_PUSH, SW41 SW_PUSH, SW42 SW_PUSH, SW43 SW_PUSH, SW44 SW_PUSH, SW45 SW_PUSH, SW46 SW_PUSH, SW47 SW_PUSH, SW48 SW_PUSH, SW49 SW_PUSH, SW5 SW_PUSH, SW50 SW_PUSH, SW51 SW_PUSH, SW52 SW_PUSH, SW53 SW_PUSH, SW54 SW_PUSH, SW55 SW_PUSH, SW56 SW_PUSH, SW57 SW_PUSH, SW58 SW_PUSH, SW59 SW_PUSH, SW6 SW_PUSH, SW60 SW_PUSH, SW61 SW_PUSH, SW62 SW_PUSH, SW63 SW_PUSH, SW64 SW_PUSH, SW65 SW_PUSH, SW7 SW_PUSH, SW8 SW_PUSH, SW9 SW_PUSH, U1 ProMicro

Commit message: Update
Parts:
- removed D16, D24, D40, D48, D49, D55, D56: D, kbd:D3_TH_SMD, symbol Device:D
- removed SW17, SW25, SW41, SW49: SW_PUSH, MXOnly:MXOnly-1U-Hotswap, symbol kbd:SW_PUSH
- removed SW50: SW_PUSH, MXOnly:MXOnly-2U-Hotswap, symbol kbd:SW_PUSH
- removed SW56: SW_PUSH, MXOnly:MXOnly-1.25U-Hotswap, symbol kbd:SW_PUSH
- removed SW57: SW_PUSH, MXOnly:MXOnly-2.75U-Hotswap-ReversedStabilizers, symbol kbd:SW_PUSH
- added D50, D59, D60, D61, D62, D63, D64, D65: D, kbd:D3_TH, symbol Device:D
- added SW33B1, SW51, SW65: SW_PUSH, MXOnly:MXOnly-1U-NoLED, symbol kbd:SW_PUSH
- added SW60, SW62, SW63, SW65B1, SW66: SW_PUSH, MXOnly:MXOnly-1.25U-NoLED, symbol kbd:SW_PUSH
- added SW61: SW_PUSH, MXOnly:MXOnly-2.75U-ReversedStabilizers-NoLED, symbol kbd:SW_PUSH
- added SW64: SW_PUSH, MXOnly:MXOnly-2.25U-ReversedStabilizers-NoLED, symbol kbd:SW_PUSH
- added SW64B1: SW_PUSH, MXOnly:MXOnly-2U-ReversedStabilizers-NoLED, symbol kbd:SW_PUSH
- D1, D10, D11, D12, D13, D14, D15, D2, D3, D4, D5, D6, D7, D8, D9: footprint kbd:D3_TH_SMD -> kbd:D3_TH
- D16: renamed from D17; footprint kbd:D3_TH_SMD -> kbd:D3_TH
- D17: renamed from D18; footprint kbd:D3_TH_SMD -> kbd:D3_TH
- D18: renamed from D19; footprint kbd:D3_TH_SMD -> kbd:D3_TH
- D19: renamed from D20; footprint kbd:D3_TH_SMD -> kbd:D3_TH
- D20: renamed from D21; footprint kbd:D3_TH_SMD -> kbd:D3_TH
- D21: renamed from D22; footprint kbd:D3_TH_SMD -> kbd:D3_TH
- D22: renamed from D23; footprint kbd:D3_TH_SMD -> kbd:D3_TH
- D23: renamed from D25; footprint kbd:D3_TH_SMD -> kbd:D3_TH
- D24: renamed from D26; footprint kbd:D3_TH_SMD -> kbd:D3_TH
- D25: renamed from D27; footprint kbd:D3_TH_SMD -> kbd:D3_TH
- D26: renamed from D28; footprint kbd:D3_TH_SMD -> kbd:D3_TH
- D27: renamed from D29; footprint kbd:D3_TH_SMD -> kbd:D3_TH
- D28: renamed from D30; footprint kbd:D3_TH_SMD -> kbd:D3_TH
- D29: renamed from D31; footprint kbd:D3_TH_SMD -> kbd:D3_TH
- D30: renamed from D32; footprint kbd:D3_TH_SMD -> kbd:D3_TH
- D31: renamed from D33; footprint kbd:D3_TH_SMD -> kbd:D3_TH
- D32: renamed from D34; footprint kbd:D3_TH_SMD -> kbd:D3_TH
- D33: renamed from D35; footprint kbd:D3_TH_SMD -> kbd:D3_TH
- D34: renamed from D36; footprint kbd:D3_TH_SMD -> kbd:D3_TH
- D35: renamed from D37; footprint kbd:D3_TH_SMD -> kbd:D3_TH
- D36: renamed from D38; footprint kbd:D3_TH_SMD -> kbd:D3_TH
- D37: renamed from D39; footprint kbd:D3_TH_SMD -> kbd:D3_TH
- D38: renamed from D41; footprint kbd:D3_TH_SMD -> kbd:D3_TH
- D39: renamed from D42; footprint kbd:D3_TH_SMD -> kbd:D3_TH
- D40: renamed from D43; footprint kbd:D3_TH_SMD -> kbd:D3_TH
- D41: renamed from D44; footprint kbd:D3_TH_SMD -> kbd:D3_TH
- D42: renamed from D45; footprint kbd:D3_TH_SMD -> kbd:D3_TH
- D43: renamed from D46; footprint kbd:D3_TH_SMD -> kbd:D3_TH
- D44: renamed from D47; footprint kbd:D3_TH_SMD -> kbd:D3_TH
- D45: renamed from D50; footprint kbd:D3_TH_SMD -> kbd:D3_TH
- D46: renamed from D51; footprint kbd:D3_TH_SMD -> kbd:D3_TH
- D47: renamed from D52; footprint kbd:D3_TH_SMD -> kbd:D3_TH
- D48: renamed from D53; footprint kbd:D3_TH_SMD -> kbd:D3_TH
- D49: renamed from D54; footprint kbd:D3_TH_SMD -> kbd:D3_TH
- D51: renamed from D57; footprint kbd:D3_TH_SMD -> kbd:D3_TH
- D52: renamed from D58; footprint kbd:D3_TH_SMD -> kbd:D3_TH
- D53: renamed from D59; footprint kbd:D3_TH_SMD -> kbd:D3_TH
- D54: renamed from D60; footprint kbd:D3_TH_SMD -> kbd:D3_TH
- D55: renamed from D61; footprint kbd:D3_TH_SMD -> kbd:D3_TH
- D56: renamed from D62; footprint kbd:D3_TH_SMD -> kbd:D3_TH
- D57: renamed from D63; footprint kbd:D3_TH_SMD -> kbd:D3_TH
- D58: renamed from D64; footprint kbd:D3_TH_SMD -> kbd:D3_TH
- SW10, SW11, SW12, SW13, SW14, SW2, SW3, SW4, SW5: footprint MXOnly:MXOnly-1U-Hotswap -> MXOnly:MXOnly-1U-NoLED
- SW15, SW6: footprint MXOnly:MXOnly-1.5U-Hotswap -> MXOnly:MXOnly-1U-NoLED
- SW16: footprint MXOnly:MXOnly-2.25U-Hotswap-ReversedStabilizers -> MXOnly:MXOnly-2U-NoLED
- SW17: renamed from SW18; footprint MXOnly:MXOnly-1U-Hotswap -> MXOnly:MXOnly-1U-NoLED
- SW18: renamed from SW19; footprint MXOnly:MXOnly-1U-Hotswap -> MXOnly:MXOnly-1.5U-NoLED
- SW19: renamed from SW20; footprint MXOnly:MXOnly-1U-Hotswap -> MXOnly:MXOnly-1U-NoLED
- SW20: renamed from SW21; footprint MXOnly:MXOnly-1U-leftleg -> MXOnly:MXOnly-1U-NoLED
- SW21: renamed from SW22; footprint MXOnly:MXOnly-1U-rightleg -> MXOnly:MXOnly-1U-NoLED
- SW22: renamed from SW23; footprint MXOnly:MXOnly-1U-Hotswap -> MXOnly:MXOnly-1U-NoLED
- SW23: renamed from SW24; footprint MXOnly:MXOnly-1U-Hotswap -> MXOnly:MXOnly-1U-NoLED
- SW24: renamed from SW26; footprint MXOnly:MXOnly-1U-Hotswap -> MXOnly:MXOnly-1U-NoLED
- SW25: renamed from SW27; footprint MXOnly:MXOnly-1U-Hotswap -> MXOnly:MXOnly-1U-NoLED
- SW26: renamed from SW28; footprint MXOnly:MXOnly-1U-Hotswap -> MXOnly:MXOnly-1U-NoLED
- SW27: renamed from SW29; footprint MXOnly:MXOnly-1U-Hotswap -> MXOnly:MXOnly-1U-NoLED
- SW28: renamed from SW30; footprint MXOnly:MXOnly-1U-Hotswap -> MXOnly:MXOnly-1U-NoLED
- SW29: renamed from SW31; footprint MXOnly:MXOnly-1U-Hotswap -> MXOnly:MXOnly-1U-NoLED
- SW30: renamed from SW32; footprint MXOnly:MXOnly-1U-Hotswap -> MXOnly:MXOnly-1U-NoLED
- SW31: renamed from SW33; footprint MXOnly:MXOnly-1U-Hotswap -> MXOnly:MXOnly-1.5U-NoLED
- SW32: renamed from SW34; footprint MXOnly:MXOnly-1U-Hotswap -> MXOnly:MXOnly-1U-NoLED
- SW33: renamed from SW35; footprint MXOnly:MXOnly-1U-Hotswap -> MXOnly:MXOnly-1.75U-NoLED
- SW34: renamed from SW36; footprint MXOnly:MXOnly-1U-Hotswap -> MXOnly:MXOnly-1U-NoLED
- SW35: renamed from SW37; footprint MXOnly:MXOnly-1U-Hotswap -> MXOnly:MXOnly-1U-NoLED
- SW36: renamed from SW38; footprint MXOnly:MXOnly-1U-Hotswap -> MXOnly:MXOnly-1U-NoLED
- SW37: renamed from SW39; footprint MXOnly:MXOnly-1U-Hotswap -> MXOnly:MXOnly-1U-NoLED
- SW38: renamed from SW40; footprint MXOnly:MXOnly-1U-Hotswap -> MXOnly:MXOnly-1U-NoLED
- SW39: renamed from SW42; footprint MXOnly:MXOnly-1U-Hotswap -> MXOnly:MXOnly-1U-NoLED
- SW40: renamed from SW43; footprint MXOnly:MXOnly-1U-Hotswap -> MXOnly:MXOnly-1U-NoLED
- SW41: renamed from SW44; footprint MXOnly:MXOnly-1U-Hotswap -> MXOnly:MXOnly-1U-NoLED
- SW42: renamed from SW45; footprint MXOnly:MXOnly-1U-Hotswap -> MXOnly:MXOnly-1U-NoLED
- SW43: renamed from SW46; footprint MXOnly:MXOnly-1U-Hotswap -> MXOnly:MXOnly-1U-NoLED
- SW44: renamed from SW47; footprint MXOnly:MXOnly-1U-Hotswap -> MXOnly:MXOnly-1U-NoLED
- SW45: renamed from SW48; footprint MXOnly:MXOnly-1U-Hotswap -> MXOnly:MXOnly-2.25U-ReversedStabilizers-NoLED
- SW46: renamed from SW51; footprint MXOnly:MXOnly-1U-Hotswap -> MXOnly:MXOnly-2.25U-NoLED
- SW47: renamed from SW52; footprint MXOnly:MXOnly-1U-Hotswap -> MXOnly:MXOnly-1U-NoLED
- SW48: renamed from SW53; footprint MXOnly:MXOnly-1U-Hotswap -> MXOnly:MXOnly-1U-NoLED
- SW49: renamed from SW54; footprint MXOnly:MXOnly-1U-Hotswap -> MXOnly:MXOnly-1U-NoLED
- SW50: renamed from SW55; footprint MXOnly:MXOnly-1U-Hotswap -> MXOnly:MXOnly-1U-NoLED
- SW52: renamed from SW58; footprint MXOnly:MXOnly-1U-Hotswap -> MXOnly:MXOnly-1U-NoLED
- SW53: renamed from SW59; footprint MXOnly:MXOnly-1U-Hotswap -> MXOnly:MXOnly-1U-NoLED
- SW54: renamed from SW60; footprint MXOnly:MXOnly-1.5U-Hotswap -> MXOnly:MXOnly-1U-NoLED
- SW55: renamed from SW61; footprint MXOnly:MXOnly-1U-Hotswap -> MXOnly:MXOnly-1U-NoLED
- SW56: renamed from SW62; footprint MXOnly:MXOnly-2.25U-Hotswap-ReversedStabilizers -> MXOnly:MXOnly-1U-NoLED
- SW57: renamed from SW63; footprint MXOnly:MXOnly-1U-Hotswap -> MXOnly:MXOnly-1U-NoLED
- SW58: renamed from SW64; footprint MXOnly:MXOnly-2.75U-Hotswap -> MXOnly:MXOnly-1.75U-NoLED
- SW59: renamed from SW65; footprint MXOnly:MXOnly-1.25U-Hotswap -> MXOnly:MXOnly-1U-NoLED
- SW7: footprint MXOnly:MXOnly-1.75U-Hotswap -> MXOnly:MXOnly-1U-NoLED
- SW8: footprint MXOnly:MXOnly-2.25U-Hotswap -> MXOnly:MXOnly-1U-NoLED
- SW9: footprint MXOnly:MXOnly-1.25U-Hotswap -> MXOnly:MXOnly-1U-NoLED
Connections:
- net col0: now also SW10.1, SW17.1, SW2.1, SW24.1, SW32.1, SW39.1, SW52.1, SW60.1
- net col1: now also SW33B1.1, SW61.1
- net col2: now also SW12.1, SW19.1, SW26.1, SW34.1, SW4.1, SW41.1, SW47.1, SW54.1, SW62.1
- net col3: now also SW13.1, SW20.1, SW27.1, SW35.1, SW42.1, SW48.1, SW5.1, SW55.1, SW63.1
- net col4: now also U1.2 (RX1/D2); no longer U1.16 (B1/15)
- net col5: now also U1.5 (2/D1/SDA), SW64.1, SW64B1.1; no longer U1.15 (B3/14)
- net col6: now also U1.6 (3/D0/SCL), SW51.1, SW65.1, SW65B1.1; no longer U1.14 (B2/16)
- net col7: now also U1.7 (4/D4), SW66.1; no longer U1.13 (B6/10)
- net row0: now also U1.8 (5/C6); no longer U1.5 (2/D1/SDA)
- net row1: now also U1.16 (B1/15); no longer U1.6 (3/D0/SCL)
- net row2: now also U1.9 (6/D7); no longer U1.7 (4/D4)
- net row3: now also U1.15 (B3/14); no longer U1.8 (5/C6)
- net row4: now also U1.10 (7/E6); no longer U1.9 (6/D7)
- net row5: now also U1.14 (B2/16); no longer U1.10 (7/E6)
- net row6: now also D50.1 (K)
- net row7: now also U1.13 (B6/10); no longer U1.12 (9/B5)
- net at D32.2 (A), SW33.2: now also SW33B1.2
- new net: D65.2 (A), SW66.2
- new net: D64.2 (A), SW65.2, SW65B1.2
- new net: D63.2 (A), SW64.2, SW64B1.2
- new net: D62.2 (A), SW63.2
- new net: D61.2 (A), SW62.2
- new net: D60.2 (A), SW61.2
- new net: D59.2 (A), SW60.2
- new net: D50.2 (A), SW51.2
- new net row8: D59.1 (K), D60.1 (K), D61.1 (K), D62.1 (K), D63.1 (K), D64.1 (K), D65.1 (K), U1.12 (9/B5)
- no-connect marks 3 -> 2
Other:
- moved on the sheet: D1, D10, D11, D12, D13, D14, D15, D16, D17, D18, D19, D2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
